File: hw/sch_pcb/ISM03.kicad_sch (KiCad schematic)
At the start: 70 parts, among them J1 JUMP_3X2, J13 HEADER_2x01_PARALLEL, J14 HEADER_2x01_PARALLEL, J15 HEADER_2x01_PARALLEL, J16 HEADER_2x01_PARALLEL, J17 HEADER_2x01_PARALLEL, J19 HEADER_2x01_PARALLEL, J2 MCX, J20 HEADER_2x01_PARALLEL, J21 HEADER_2x01_PARALLEL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

Commit message: Update documentation PCB WiP.
Parts:
- added R2, R3: 1k, Resistor_SMD:R_0805_2012Metric, symbol Device:R
- C1, C10, C12, C13, C15, C17, C19, C2, C20, C3, C4, C5, C6, C7, C8, C9: footprint Mlab_R:SMD-0805 -> Capacitor_SMD:C_0805_2012Metric
- D1: footprint Mlab_D:Diode-MiniMELF_Standard -> Diode_SMD:D_SMA
- R1: value 0R -> 3R; UST_ID 5c70984512875079b91f896b -> 60d57f1a1287500165f858ae
Connections:
- net at C13.1, L10.1, L9.2: now also U2.2 (RXp); no longer U2.3 (RXn)
- net at C12.1, L10.2: now also U2.3 (RXn); no longer U2.2 (RXp)
- net at Q1.1 (B): now also R2.2; no longer J24.1
- net at Q2.1 (B): now also R3.2; no longer J25.1
- new net: J25.1, R3.1
- new net: J24.1, R2.1
Other:
- moved on the sheet: D2, J24, J25, Q1, R22

Commit message: Backup work before switching to KiCADv8
Parts:
- added J5: HEADER_2x01_PARALLEL, Mlab_Pin_Headers:Straight_2x01, symbol MLAB_HEADER:HEADER_2x01_PARALLEL
- added R4: 33R, Resistor_SMD:R_0805_2012Metric, symbol Device:R
- added R5: 10k, Resistor_SMD:R_0805_2012Metric, symbol Device:R
- R2, R3: value 1k -> 10k
Connections:
- net GND: now also R5.1
- net at U2.1 (SDN): now also R4.2
- new net SDN: J5.1, J5.2, R4.1, R5.2
Other:
- moved on the sheet: C15, C17, C19, C20, L11
